File: ProgNRF52/Prog_NRF52.brd (EAGLE design)
At the start: 46.8 x 66.4 mm, 48 parts, among them J3 MEC1-108-02-XX-D-A, U1 TS5A9411, U2 SN74LVC1GU04DBV, U3 TS5A9411, U4 TS5A9411, U5 SN74LVC1GU04DBV, U6 TXB0102D

Commit message: Change layout
Changing current layout
Parts:
- moved C10 116.2 mm to (58.5, 46.9)
- moved C6 116.2 mm to (58.5, 63.7)
- moved C7 116.2 mm to (58.5, 59.5)
- moved C8 116.2 mm to (58.5, 55.3)
- moved C9 116.2 mm to (58.5, 51.1)
- moved R10 116.2 mm to (58.6, 32.8)
- moved R6 116.2 mm to (58.6, 68.2)
- moved R7 116.2 mm to (58.6, 42.4)
- moved R9 116.2 mm to (58.6, 37.6)
- moved U7 76.8 mm to (49.2, 44.4)
- moved U6 68.6 mm to (49.2, 38.7)
Changed lines of the file:
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@@
 <attribute name="VALUE" x="14.19" y="57.779" size="1.27" layer="27" ratio="10"/>
 </element>
-<element name="U6" library="Tmp_PN" package="VSSOP8" value="TXB0102D" x="-6.7" y="-1"/>
-<element name="U7" library="Tmp_PN" package="SOT23-5" value="" x="-13.3" y="-0.3"/>
+<element name="U6" library="Tmp_PN" package="VSSOP8" value="TXB0102D" x="49.2" y="38.7"/>
+<element name="U7" library="Tmp_PN" package="SOT23-5" value="" x="49.2" y="44.4"/>
 <element name="TP1" library="testpad" package="P1-13" value="TPPAD1-13" x="38.2" y="74.8">
 <attribute name="TP_SIGNAL_NAME" value="" x="38.2" y="74.8" size="1.778" layer="27" display="off"/>
@@
 <attribute name="TP_SIGNAL_NAME" value="" x="51.2" y="75" size="1.778" layer="27" display="off"/>
 </element>
-<element name="R6" library="resistor" package="R0603" value="NC" x="-14.2" y="-22.4"/>
-<element name="C6" library="rcl" package="C0603K" value="1uF" x="-14.3" y="-26.9"/>
-<element name="C7" library="rcl" package="C0603K" value="1uF" x="-14.3" y="-31.1"/>
-<element name="C8" library="rcl" package="C0603K" value="100nF" x="-14.3" y="-35.3"/>
-<element name="C9" library="rcl" package="C0603K" value="100nF" x="-14.3" y="-39.5"/>
-<element name="C10" library="rcl" package="C0603K" value="100nF" x="-14.3" y="-43.7"/>
-<element name="R7" library="resistor" package="R0603" value="10K" x="-14.2" y="-48.2"/>
-<element name="R9" library="resistor" package="R0603" value="NC" x="-14.2" y="-53"/>
-<element name="R10" library="resistor" package="R0603" value="NC" x="-14.2" y="-57.8"/>
+<element name="R6" library="resistor" package="R0603" value="NC" x="58.6" y="68.2"/>
+<element name="C6" library="rcl" package="C0603K" value="1uF" x="58.5" y="63.7"/>
+<element name="C7" library="rcl" package="C0603K" value="1uF" x="58.5" y="59.5"/>
+<element name="C8" library="rcl" package="C0603K" value="100nF" x="58.5" y="55.3"/>
+<element name="C9" library="rcl" package="C0603K" value="100nF" x="58.5" y="51.1"/>
+<element name="C10" library="rcl" package="C0603K" value="100nF" x="58.5" y="46.9"/>
+<element name="R7" library="resistor" package="R0603" value="10K" x="58.6" y="42.4"/>
+<element name="R9" library="resistor" package="R0603" value="NC" x="58.6" y="37.6"/>
+<element name="R10" library="resistor" package="R0603" value="NC" x="58.6" y="32.8"/>
 </elements>
 <signals>
@@
 <contactref element="C10" pad="2"/>
 <contactref element="TP4" pad="TP"/>
-<wire x1="-15.175" y1="-39.5" x2="-13.425" y2="-43.7" width="0" layer="19" extent="1-1"/>
-<wire x1="-13.425" y1="-35.3" x2="-15.175" y2="-39.5" width="0" layer="19" extent="1-1"/>
-<wire x1="-15.175" y1="-31.1" x2="-13.425" y2="-35.3" width="0" layer="19" extent="1-1"/>
-<wire x1="-15.175" y1="-26.9" x2="-15.175" y2="-31.1" width="0" layer="19" extent="1-1"/>
-<wire x1="51.2" y1="75" x2="-15.175" y2="-26.9" width="0" layer="19" extent="1-1"/>
-<wire x1="-7.025" y1="-3.325" x2="51.2" y2="75" width="0" layer="19" extent="1-1"/>
-<wire x1="-13.3" y1="-1.6001" x2="-7.025" y2="-3.325" width="0" layer="19" extent="1-1"/>
-<wire x1="13.1" y1="7.59" x2="-7.025" y2="-3.325" width="0" layer="19" extent="1-1"/>
+<wire x1="57.625" y1="51.1" x2="59.375" y2="46.9" width="0" layer="19" extent="1-1"/>
+<wire x1="59.375" y1="55.3" x2="57.625" y2="51.1" width="0" layer="19" extent="1-1"/>
+<wire x1="57.625" y1="59.5" x2="59.375" y2="55.3" width="0" layer="19" extent="1-1"/>
+<wire x1="57.625" y1="63.7" x2="57.625" y2="59.5" width="0" layer="19" extent="1-1"/>
+<wire x1="51.2" y1="75" x2="57.625" y2="63.7" width="0" layer="19" extent="1-1"/>
+<wire x1="48.875" y1="36.375" x2="51.2" y2="75" width="0" layer="19" extent="1-1"/>
+<wire x1="49.2" y1="43.0999" x2="48.875" y2="36.375" width="0" layer="19" extent="1-1"/>
+<wire x1="13.1" y1="7.59" x2="48.875" y2="36.375" width="0" layer="19" extent="1-1"/>
 </signal>
 <signal name="+5V">
@@
 <contactref element="C8" pad="1"/>
 <wire x1="47.6" y1="11.91" x2="47.55" y2="11.86" width="0" layer="19" extent="1-1"/>
-<wire x1="-7.025" y1="1.325" x2="27.2" y2="12.7" width="0" layer="19" extent="1-16"/>
-<wire x1="-12.35" y1="-1.6001" x2="-7.025" y2="1.325" width="0" layer="19" extent="1-1"/>
-<wire x1="-14.25" y1="-1.6001" x2="-12.35" y2="-1.6001" width="0" layer="19" extent="1-1"/>
-<wire x1="-13.425" y1="-26.9" x2="-14.25" y2="-1.6001" width="0" layer="19" extent="1-1"/>
-<wire x1="-15.175" y1="-35.3" x2="-13.425" y2="-26.9" width="0" layer="19" extent="1-1"/>
+<wire x1="48.875" y1="41.025" x2="27.2" y2="12.7" width="0" layer="19" extent="1-16"/>
+<wire x1="50.15" y1="43.0999" x2="48.875" y2="41.025" width="0" layer="19" extent="1-1"/>
+<wire x1="48.25" y1="43.0999" x2="50.15" y2="43.0999" width="0" layer="19" extent="1-1"/>
+<wire x1="59.375" y1="63.7" x2="48.25" y2="43.0999" width="0" layer="19" extent="1-1"/>
+<wire x1="57.625" y1="55.3" x2="59.375" y2="63.7" width="0" layer="19" extent="1-1"/>
 </signal>
 <signal name="RESET">
@@
 <wire x1="15.6" y1="51.9" x2="21.7" y2="58" width="0.3" layer="1"/>
 <contactref element="R6" pad="2"/>
-<wire x1="-13.35" y1="-22.4" x2="21.1" y2="16.6" width="0" layer="19" extent="1-1"/>
+<wire x1="59.45" y1="68.2" x2="21.1" y2="16.6" width="0" layer="19" extent="1-1"/>
 </signal>
 <signal name="N$8">
@@
 <contactref element="TP2" pad="TP"/>
 <contactref element="R9" pad="2"/>
-<wire x1="42.1" y1="74.8" x2="-13.35" y2="-53" width="0" layer="19" extent="1-1"/>
-<wire x1="-5.725" y1="1.325" x2="42.1" y2="74.8" width="0" layer="19" extent="1-1"/>
-<wire x1="24.8" y1="29.5" x2="-5.725" y2="1.325" width="0" layer="19" extent="1-1"/>
+<wire x1="42.1" y1="74.8" x2="59.45" y2="37.6" width="0" layer="19" extent="1-1"/>
+<wire x1="50.175" y1="41.025" x2="42.1" y2="74.8" width="0" layer="19" extent="1-1"/>
+<wire x1="24.8" y1="29.5" x2="50.175" y2="41.025" width="0" layer="19" extent="1-1"/>
 </signal>
 <signal name="SWDIO">
@@
 <contactref element="U6" pad="1"/>
 <contactref element="R10" pad="1"/>
-<wire x1="-7.675" y1="-3.325" x2="-15.05" y2="-57.8" width="0" layer="19" extent="1-1"/>
-<wire x1="36.2" y1="27.3" x2="-7.675" y2="-3.325" width="0" layer="19" extent="1-1"/>
+<wire x1="48.225" y1="36.375" x2="57.75" y2="32.8" width="0" layer="19" extent="1-1"/>
+<wire x1="36.2" y1="27.3" x2="48.225" y2="36.375" width="0" layer="19" extent="1-1"/>
 </signal>
 <signal name="PN_UART_TXD">
@@
 <contactref element="R6" pad="1"/>
 <contactref element="CONN1" pad="1"/>
-<wire x1="-15.05" y1="-22.4" x2="28.04" y2="53.132" width="0" layer="19" extent="1-1"/>
+<wire x1="57.75" y1="68.2" x2="28.04" y2="53.132" width="0" layer="19" extent="1-1"/>
 </signal>
 <signal name="+2V8">
@@
 <contactref element="C9" pad="2"/>
 <contactref element="R7" pad="2"/>
-<wire x1="-13.425" y1="-39.5" x2="-13.35" y2="-48.2" width="0" layer="19" extent="1-1"/>
-<wire x1="-13.425" y1="-31.1" x2="-13.425" y2="-39.5" width="0" layer="19" extent="1-1"/>
-<wire x1="-6.375" y1="-3.325" x2="-13.425" y2="-31.1" width="0" layer="19" extent="1-1"/>
-<wire x1="-14.25" y1="1.0001" x2="-6.375" y2="-3.325" width="0" layer="19" extent="1-1"/>
+<wire x1="59.375" y1="51.1" x2="59.45" y2="42.4" width="0" layer="19" extent="1-1"/>
+<wire x1="59.375" y1="59.5" x2="59.375" y2="51.1" width="0" layer="19" extent="1-1"/>
+<wire x1="49.525" y1="36.375" x2="59.375" y2="59.5" width="0" layer="19" extent="1-1"/>
+<wire x1="48.25" y1="45.7001" x2="49.525" y2="36.375" width="0" layer="19" extent="1-1"/>
 </signal>
 <signal name="SWDCLK">
@@
 <contactref element="U6" pad="8"/>
 <contactref element="R9" pad="1"/>
-<wire x1="-7.675" y1="1.325" x2="-15.05" y2="-53" width="0" layer="19" extent="1-1"/>
-<wire x1="29.89" y1="23.48" x2="-7.675" y2="1.325" width="0" layer="19" extent="1-1"/>
+<wire x1="48.225" y1="41.025" x2="57.75" y2="37.6" width="0" layer="19" extent="1-1"/>
+<wire x1="29.89" y1="23.48" x2="48.225" y2="41.025" width="0" layer="19" extent="1-1"/>
 </signal>
 <signal name="PN_SWDIO">
@@
 <contactref element="R10" pad="2"/>
 <wire x1="28.04" y1="49.068" x2="31.3" y2="61.0695" width="0" layer="19" extent="1-1"/>
-<wire x1="-5.725" y1="-3.325" x2="28.04" y2="49.068" width="0" layer="19" extent="1-1"/>
-<wire x1="38.2" y1="74.8" x2="-5.725" y2="-3.325" width="0" layer="19" extent="1-1"/>
-<wire x1="-13.35" y1="-57.8" x2="38.2" y2="74.8" width="0" layer="19" extent="1-1"/>
+<wire x1="50.175" y1="36.375" x2="28.04" y2="49.068" width="0" layer="19" extent="1-1"/>
+<wire x1="38.2" y1="74.8" x2="50.175" y2="36.375" width="0" layer="19" extent="1-1"/>
+<wire x1="59.45" y1="32.8" x2="38.2" y2="74.8" width="0" layer="19" extent="1-1"/>
 </signal>
 <signal name="N$27">
@@
 <contactref element="U6" pad="6"/>
 <contactref element="C10" pad="1"/>
-<wire x1="-15.175" y1="-43.7" x2="-15.05" y2="-48.2" width="0" layer="19" extent="1-1"/>
-<wire x1="-6.375" y1="1.325" x2="-15.175" y2="-43.7" width="0" layer="19" extent="1-1"/>
+<wire x1="57.625" y1="46.9" x2="57.75" y2="42.4" width="0" layer="19" extent="1-1"/>
+<wire x1="49.525" y1="41.025" x2="57.625" y2="46.9" width="0" layer="19" extent="1-1"/>
 </signal>
 </signals>

Commit message: update schematic comments
update schematic and layout
Parts:
- removed LED2: (no value), led:CHIP-LED0603
- removed R3: 220, resistor:R0603
- moved R10 8.92 mm to (49.7, 33.4)
- moved TP3 7.21 mm to (47.2, 67.8)
- moved TP2 7.16 mm to (43.6, 67.8)
- moved TP1 7.12 mm to (39.5, 67.8)
- moved TP4 7.12 mm to (50.7, 67.9)
Connections:
- removed net N$4: LED2.C, R3.2
- net FT_SWD_OE: no longer LED2.A
- net GND: no longer R3.1
Routing:
- net N$4: track 1.50 -> 0.00 mm
- net FT_SWD_OE: track 43.1 -> 42.0 mm
Changed lines of the file:
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@@
 </element>
 <element name="R4" library="resistor" package="R0603" value="470" x="8.99" y="51.62" smashed="yes" rot="R270">
-<attribute name="NAME" x="8.425" y="58.455" size="1.27" layer="25" rot="R270"/>
+<attribute name="NAME" x="8.425" y="58.155" size="1.27" layer="25" rot="R270"/>
 <attribute name="VALUE" x="8.585" y="55.155" size="1" layer="27" rot="R270"/>
 </element>
 <element name="R5" library="resistor" package="R0603" value="470" x="11.14" y="51.61" smashed="yes" rot="R270">
-<attribute name="NAME" x="10.575" y="58.445" size="1.27" layer="25" rot="R270"/>
+<attribute name="NAME" x="10.675" y="58.145" size="1.27" layer="25" rot="R270"/>
 <attribute name="VALUE" x="10.735" y="55.045" size="1" layer="27" rot="R270"/>
 </element>
@@
 </element>
 <element name="U1" library="FabLib" package="SC70-6" value="TS5A9411" x="45.76" y="29.12" smashed="yes" rot="R90">
-<attribute name="NAME" x="44.3312" y="27.85" size="1.016" layer="25" ratio="18" rot="R90"/>
+<attribute name="NAME" x="46.65" y="31.7312" size="1.016" layer="25" ratio="18" rot="R180"/>
 <attribute name="VALUE" x="48.05" y="31.6825" size="0.8128" layer="27" ratio="10" rot="R180"/>
 </element>
@@
 </element>
 <element name="CONN1" library="con-Samtec" package="FTS-105-01-F-DV" value="FTS-105-01-F-DV" x="25.5" y="51.1" smashed="yes" rot="R270">
-<attribute name="NAME" x="20.395" y="53.6" size="1.27" layer="25" rot="R270"/>
+<attribute name="NAME" x="20.595" y="51.8" size="1.27" layer="25" rot="R270"/>
 <attribute name="VALUE" x="20.135" y="46.575" size="1" layer="27"/>
 </element>
@@
 <attribute name="VALUE" x="42.41" y="47.921" size="1.27" layer="27" ratio="10" rot="R180"/>
 </element>
-<element name="LED2" library="led" package="CHIP-LED0603" value="" x="45.8" y="48.3" smashed="yes">
-<attribute name="NAME" x="46.165" y="43.665" size="1" layer="25" rot="R90"/>
-<attribute name="VALUE" x="47.705" y="47.665" size="1.27" layer="27" rot="R90"/>
-</element>
-<element name="R3" library="resistor" package="R0603" value="220" x="45.8" y="51.4" smashed="yes" rot="R270">
-<attribute name="NAME" x="45.135" y="54.635" size="1.27" layer="25" rot="R270"/>
-<attribute name="VALUE" x="45.395" y="54.835" size="1" layer="27" rot="R270"/>
-</element>
 <element name="J3" library="TestBench_MUX" package="MEC1-108-02-XX-D-A" value="MEC1-108-02-XX-D-A" x="28.8" y="64.6" smashed="yes">
 <attribute name="NAME" x="36" y="68.2" size="1.27" layer="25"/>
@@
 <element name="U6" library="Tmp_PN" package="VSSOP8" value="TXB0102D" x="49.2" y="38.7"/>
 <element name="U7" library="Tmp_PN" package="SOT23-5" value="" x="49.2" y="44.4"/>
-<element name="TP1" library="testpad" package="P1-13" value="TPPAD1-13" x="38.2" y="74.8">
-<attribute name="TP_SIGNAL_NAME" value="" x="38.2" y="74.8" size="1.778" layer="27" display="off"/>
-</element>
-<element name="TP2" library="testpad" package="P1-13" value="TPPAD1-13" x="42.1" y="74.8">
-<attribute name="TP_SIGNAL_NAME" value="" x="42.1" y="74.8" size="1.778" layer="27" display="off"/>
-</element>
-<element name="TP3" library="testpad" package="P1-13" value="TPPAD1-13" x="46.8" y="75">
-<attribute name="TP_SIGNAL_NAME" value="" x="46.8" y="75" size="1.778" layer="27" display="off"/>
-</element>
-<element name="TP4" library="testpad" package="P1-13" value="TPPAD1-13" x="51.2" y="75">
-<attribute name="TP_SIGNAL_NAME" value="" x="51.2" y="75" size="1.778" layer="27" display="off"/>
+<element name="TP1" library="testpad" package="P1-13" value="TPPAD1-13" x="39.5" y="67.8">
+<attribute name="TP_SIGNAL_NAME" value="" x="39.5" y="67.8" size="1.778" layer="27" display="off"/>
+</element>
+<element name="TP2" library="testpad" package="P1-13" value="TPPAD1-13" x="43.6" y="67.8">
+<attribute name="TP_SIGNAL_NAME" value="" x="43.6" y="67.8" size="1.778" layer="27" display="off"/>
+</element>
+<element name="TP3" library="testpad" package="P1-13" value="TPPAD1-13" x="47.2" y="67.8">
+<attribute name="TP_SIGNAL_NAME" value="" x="47.2" y="67.8" size="1.778" layer="27" display="off"/>
+</element>
+<element name="TP4" library="testpad" package="P1-13" value="TPPAD1-13" x="50.7" y="67.9">
+<attribute name="TP_SIGNAL_NAME" value="" x="50.7" y="67.9" size="1.778" layer="27" display="off"/>
 </element>
 <element name="R6" library="resistor" package="R0603" value="NC" x="58.6" y="68.2"/>
@@
 <element name="R7" library="resistor" package="R0603" value="10K" x="58.6" y="42.4"/>
 <element name="R9" library="resistor" package="R0603" value="NC" x="58.6" y="37.6"/>
-<element name="R10" library="resistor" package="R0603" value="NC" x="58.6" y="32.8"/>
+<element name="R10" library="resistor" package="R0603" value="NC" x="49.7" y="33.4" smashed="yes">
+<attribute name="NAME" x="51.365" y="32.835" size="1.27" layer="25"/>
+<attribute name="VALUE" x="49.065" y="31.495" size="1.27" layer="27"/>
+</element>
 </elements>
 <signals>
@@
 <contactref element="C5" pad="1"/>
 <contactref element="J4" pad="1"/>
-<contactref element="R3" pad="1"/>
 <wire x1="25.5" y1="53.132" x2="25.5" y2="55.4" width="0.3" layer="1"/>
 <wire x1="25.5" y1="55.4" x2="25.6" y2="55.5" width="0.3" layer="1"/>
@@
 <wire x1="26.1" y1="53.1" x2="26.2" y2="53.2" width="0.3" layer="16"/>
 <wire x1="43.39" y1="52.21" x2="45.76" y2="52.21" width="0.3" layer="1"/>
-<wire x1="45.76" y1="52.21" x2="45.8" y2="52.25" width="0.3" layer="1"/>
 <wire x1="43.39" y1="52.21" x2="41.71" y2="52.21" width="0.3" layer="1"/>
 <wire x1="41.71" y1="52.21" x2="41.7" y2="52.2" width="0.3" layer="1"/>
@@
 <contactref element="C10" pad="2"/>
 <contactref element="TP4" pad="TP"/>
-<wire x1="57.625" y1="51.1" x2="59.375" y2="46.9" width="0" layer="19" extent="1-1"/>
-<wire x1="59.375" y1="55.3" x2="57.625" y2="51.1" width="0" layer="19" extent="1-1"/>
-<wire x1="57.625" y1="59.5" x2="59.375" y2="55.3" width="0" layer="19" extent="1-1"/>
-<wire x1="57.625" y1="63.7" x2="57.625" y2="59.5" width="0" layer="19" extent="1-1"/>
-<wire x1="51.2" y1="75" x2="57.625" y2="63.7" width="0" layer="19" extent="1-1"/>
-<wire x1="48.875" y1="36.375" x2="51.2" y2="75" width="0" layer="19" extent="1-1"/>
-<wire x1="49.2" y1="43.0999" x2="48.875" y2="36.375" width="0" layer="19" extent="1-1"/>
-<wire x1="13.1" y1="7.59" x2="48.875" y2="36.375" width="0" layer="19" extent="1-1"/>
+<wire x1="57.625" y1="59.5" x2="57.625" y2="63.7" width="0" layer="19" extent="1-1"/>
+<wire x1="59.375" y1="55.3" x2="57.625" y2="59.5" width="0" layer="19" extent="1-1"/>
+<wire x1="57.625" y1="51.1" x2="59.375" y2="55.3" width="0" layer="19" extent="1-1"/>
+<wire x1="59.375" y1="46.9" x2="57.625" y2="51.1" width="0" layer="19" extent="1-1"/>
+<wire x1="50.7" y1="67.9" x2="57.625" y2="63.7" width="0" layer="19" extent="1-1"/>
+<wire x1="49.2" y1="43.0999" x2="59.375" y2="46.9" width="0" layer="19" extent="1-1"/>
+<wire x1="45.5" y1="40.6" x2="49.2" y2="43.0999" width="0" layer="19" extent="1-16"/>
+<wire x1="48.875" y1="36.375" x2="45.5" y2="34.7" width="0" layer="19" extent="1-16"/>
 </signal>
 <signal name="+5V">
@@
 <wire x1="30.3" y1="61.0695" x2="30.3" y2="51.1" width="0.3" layer="1"/>
 <contactref element="TP3" pad="TP"/>
-<wire x1="46.8" y1="75" x2="22.96" y2="49.068" width="0" layer="19" extent="1-1"/>
+<wire x1="47.2" y1="67.8" x2="22.96" y2="49.068" width="0" layer="19" extent="1-1"/>
 </signal>
 <signal name="SWD_EN">
@@
 <wire x1="26" y1="40.8" x2="25.9" y2="40.7" width="0.3" layer="16"/>
 </signal>
-<signal name="N$4">
-<contactref element="LED2" pad="C"/>
-<contactref element="R3" pad="2"/>
-<wire x1="45.8" y1="50.55" x2="45.8" y2="49.05" width="0.3" layer="1"/>
-</signal>
 <signal name="N$5">
 <wire x1="45.607" y1="64.666" x2="47.385" y2="64.666" width="0.254" layer="1"/>
@@
 <wire x1="33.56" y1="30.55" x2="33.51" y2="30.5" width="0.3" layer="16"/>
 <contactref element="U1" pad="1"/>
-<contactref element="LED2" pad="A"/>
 <wire x1="46.93" y1="28.47" x2="48.1" y2="27.3" width="0.3" layer="1"/>
 <wire x1="48.1" y1="27.3" x2="50.5" y2="27.3" width="0.3" layer="1"/>
@@
 <wire x1="46.93" y1="28.47" x2="46.71" y2="28.47" width="0.3" layer="1"/>
 <wire x1="45.5" y1="30.9" x2="39.05" y2="30.9" width="0.3" layer="1"/>
-<wire x1="45.8" y1="46.4" x2="45.8" y2="47.55" width="0.3" layer="1"/>
 <wire x1="47.2" y1="31.8" x2="47.2" y2="45" width="0.3" layer="1"/>
 <wire x1="47.2" y1="45" x2="45.8" y2="46.4" width="0.3" layer="1"/>
@@
 <contactref element="TP2" pad="TP"/>
 <contactref element="R9" pad="2"/>
-<wire x1="42.1" y1="74.8" x2="59.45" y2="37.6" width="0" layer="19" extent="1-1"/>
-<wire x1="50.175" y1="41.025" x2="42.1" y2="74.8" width="0" layer="19" extent="1-1"/>
+<wire x1="43.6" y1="67.8" x2="59.45" y2="37.6" width="0" layer="19" extent="1-1"/>
+<wire x1="50.175" y1="41.025" x2="43.6" y2="67.8" width="0" layer="19" extent="1-1"/>
 <wire x1="24.8" y1="29.5" x2="50.175" y2="41.025" width="0" layer="19" extent="1-1"/>
 </signal>
@@
 <contactref element="U6" pad="1"/>
 <contactref element="R10" pad="1"/>
-<wire x1="48.225" y1="36.375" x2="57.75" y2="32.8" width="0" layer="19" extent="1-1"/>
+<wire x1="48.225" y1="36.375" x2="48.85" y2="33.4" width="0" layer="19" extent="1-1"/>
 <wire x1="36.2" y1="27.3" x2="48.225" y2="36.375" width="0" layer="19" extent="1-1"/>
 </signal>
@@
 <wire x1="28.04" y1="49.068" x2="31.3" y2="61.0695" width="0" layer="19" extent="1-1"/>
 <wire x1="50.175" y1="36.375" x2="28.04" y2="49.068" width="0" layer="19" extent="1-1"/>
-<wire x1="38.2" y1="74.8" x2="50.175" y2="36.375" width="0" layer="19" extent="1-1"/>
-<wire x1="59.45" y1="32.8" x2="38.2" y2="74.8" width="0" layer="19" extent="1-1"/>
+<wire x1="39.5" y1="67.8" x2="50.175" y2="36.375" width="0" layer="19" extent="1-1"/>
+<wire x1="50.55" y1="33.4" x2="39.5" y2="67.8" width="0" layer="19" extent="1-1"/>
 </signal>
 <signal name="N$27">
