File: ProgNRF52/Prog_NRF52.brd (EAGLE design)
At the start: 46.8 x 66.4 mm, 46 parts, among them J3 MEC1-108-02-XX-D-A, U1 TS5A9411, U2 SN74LVC1GU04DBV, U3 TS5A9411, U4 TS5A9411, U5 SN74LVC1GU04DBV, U6 TXB0102D

Commit message: Suppress led on schematic
Useless led where suppress
Parts:
- removed LED4: (no value), led:CHIP-LED0603
- removed R5: 470, resistor:R0603
Connections:
- removed net N$7: LED4.A, R5.2
- net +3V3: no longer R5.1
- net RX_LED: no longer LED4.C
Routing:
- net RX_LED: track 13.3 -> 7.63 mm
- net N$7: track 1.65 -> 0.00 mm
Changed lines of the file:
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@@
 <attribute name="VALUE" x="7.185" y="49.015" size="1.27" layer="27" rot="R270"/>
-</element>
-<element name="LED4" library="led" package="CHIP-LED0603" value="" x="11.2" y="48.38" smashed="yes" rot="R180">
-<attribute name="NAME" x="10.835" y="46.915" size="1.27" layer="25" rot="R270"/>
-<attribute name="VALUE" x="9.295" y="49.015" size="1.27" layer="27" rot="R270"/>
 </element>
 <element name="R1" library="resistor" package="R0603" value="nc" x="44.9" y="26.76" smashed="yes" rot="R180">
@@
 <attribute name="NAME" x="8.425" y="58.155" size="1.27" layer="25" rot="R270"/>
 <attribute name="VALUE" x="8.585" y="55.155" size="1" layer="27" rot="R270"/>
-</element>
-<element name="R5" library="resistor" package="R0603" value="470" x="11.14" y="51.61" smashed="yes" rot="R270">
-<attribute name="NAME" x="10.675" y="58.145" size="1.27" layer="25" rot="R270"/>
-<attribute name="VALUE" x="10.735" y="55.045" size="1" layer="27" rot="R270"/>
 </element>
 <element name="JMP4" library="con-lstb" package="MA02-1" value="" x="8.34" y="10.09" rot="R270"/>
@@
 <contactref element="U1" pad="2"/>
 <contactref element="R4" pad="1"/>
-<contactref element="R5" pad="1"/>
 <contactref element="C4" pad="1"/>
 <contactref element="U5" pad="5"/>
@@
 <wire x1="8.97" y1="52.45" x2="8.99" y2="52.47" width="0.3" layer="1"/>
 <wire x1="8.99" y1="52.47" x2="11.13" y2="52.47" width="0.3" layer="1"/>
-<wire x1="11.13" y1="52.47" x2="11.14" y2="52.46" width="0.3" layer="1"/>
 <wire x1="8.99" y1="52.47" x2="8.99" y2="53.99" width="0.3" layer="1"/>
 <wire x1="8.99" y1="53.99" x2="9" y2="54" width="0.3" layer="1"/>
@@
 <contactref element="U6" pad="7"/>
 <contactref element="C8" pad="1"/>
-<wire x1="47.6" y1="11.91" x2="47.55" y2="11.86" width="0" layer="19" extent="1-1"/>
-<wire x1="48.875" y1="41.025" x2="27.2" y2="12.7" width="0" layer="19" extent="1-16"/>
-<wire x1="50.15" y1="43.0999" x2="48.875" y2="41.025" width="0" layer="19" extent="1-1"/>
+<wire x1="57.625" y1="55.3" x2="59.375" y2="63.7" width="0" layer="19" extent="1-1"/>
+<wire x1="50.15" y1="43.0999" x2="57.625" y2="55.3" width="0" layer="19" extent="1-1"/>
 <wire x1="48.25" y1="43.0999" x2="50.15" y2="43.0999" width="0" layer="19" extent="1-1"/>
-<wire x1="59.375" y1="63.7" x2="48.25" y2="43.0999" width="0" layer="19" extent="1-1"/>
-<wire x1="57.625" y1="55.3" x2="59.375" y2="63.7" width="0" layer="19" extent="1-1"/>
+<wire x1="48.875" y1="41.025" x2="48.25" y2="43.0999" width="0" layer="19" extent="1-1"/>
+<wire x1="48" y1="30.2" x2="48.875" y2="41.025" width="0" layer="19" extent="1-1"/>
+<wire x1="47.55" y1="11.86" x2="47.6" y2="11.91" width="0" layer="19" extent="1-1"/>
 </signal>
 <signal name="RESET">
@@
 <wire x1="9" y1="49.22" x2="9.09" y2="49.13" width="0.3" layer="1"/>
 </signal>
-<signal name="N$7">
-<contactref element="LED4" pad="A"/>
-<contactref element="R5" pad="2"/>
-<wire x1="11.14" y1="50.76" x2="11.14" y2="49.19" width="0.3" layer="1"/>
-<wire x1="11.14" y1="49.19" x2="11.2" y2="49.13" width="0.3" layer="1"/>
-</signal>
 <signal name="VTG">
 <contactref element="J2" pad="2"/>
@@
 <contactref element="J4" pad="14"/>
 <contactref element="J1" pad="14"/>
-<contactref element="LED4" pad="C"/>
 <wire x1="13.01" y1="40.7" x2="13.1" y2="40.61" width="0.3" layer="1"/>
 <wire x1="18.23" y1="40.66" x2="13.15" y2="40.66" width="0.3" layer="16"/>
@@
 <wire x1="13.01" y1="40.7" x2="12.5" y2="40.7" width="0.3" layer="1"/>
 <wire x1="12.5" y1="40.7" x2="11.2" y2="42" width="0.3" layer="1"/>
-<wire x1="11.2" y1="42" x2="11.2" y2="47.63" width="0.3" layer="1"/>
 </signal>
 <signal name="N$19">

Commit message: Test : remove voltage translation unit
Remove to test revory sch
Parts:
- removed C10, C8, C9: 100nF, rcl:C0603K
- removed R7: 10K, resistor:R0603
- removed U6: TXB0102D, Tmp_PN:VSSOP8
Connections:
- removed net N$27: C10.1, R7.1, U6.6
- net +2V8: no longer C9.2, R7.2, U6.3
- net +3V3: no longer C8.1, U6.7
- net GND: no longer C10.2, C8.2, C9.1, U6.2
- net PN_SWDCLK: no longer U6.5
- net PN_SWDIO: no longer U6.4
- net SWDCLK: no longer U6.8
- net SWDIO: no longer U6.1
Changed lines of the file:
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@@
 <attribute name="VALUE" x="14.19" y="57.779" size="1.27" layer="27" ratio="10"/>
 </element>
-<element name="U6" library="Tmp_PN" package="VSSOP8" value="TXB0102D" x="49.2" y="38.7"/>
 <element name="U7" library="Tmp_PN" package="SOT23-5" value="" x="49.2" y="44.4"/>
 <element name="TP1" library="testpad" package="P1-13" value="TPPAD1-13" x="39.5" y="67.8">
@@
 <element name="C6" library="rcl" package="C0603K" value="1uF" x="58.5" y="63.7"/>
 <element name="C7" library="rcl" package="C0603K" value="1uF" x="58.5" y="59.5"/>
-<element name="C8" library="rcl" package="C0603K" value="100nF" x="58.5" y="55.3"/>
-<element name="C9" library="rcl" package="C0603K" value="100nF" x="58.5" y="51.1"/>
-<element name="C10" library="rcl" package="C0603K" value="100nF" x="58.5" y="46.9"/>
-<element name="R7" library="resistor" package="R0603" value="10K" x="58.6" y="42.4"/>
 <element name="R9" library="resistor" package="R0603" value="NC" x="58.6" y="37.6"/>
 <element name="R10" library="resistor" package="R0603" value="NC" x="49.7" y="33.4" smashed="yes">
@@
 <contactref element="C7" pad="1"/>
 <contactref element="C6" pad="1"/>
-<contactref element="U6" pad="2"/>
-<contactref element="C8" pad="2"/>
-<contactref element="C9" pad="1"/>
-<contactref element="C10" pad="2"/>
 <contactref element="TP4" pad="TP"/>
 <wire x1="57.625" y1="59.5" x2="57.625" y2="63.7" width="0" layer="19" extent="1-1"/>
-<wire x1="59.375" y1="55.3" x2="57.625" y2="59.5" width="0" layer="19" extent="1-1"/>
-<wire x1="57.625" y1="51.1" x2="59.375" y2="55.3" width="0" layer="19" extent="1-1"/>
-<wire x1="59.375" y1="46.9" x2="57.625" y2="51.1" width="0" layer="19" extent="1-1"/>
 <wire x1="50.7" y1="67.9" x2="57.625" y2="63.7" width="0" layer="19" extent="1-1"/>
-<wire x1="49.2" y1="43.0999" x2="59.375" y2="46.9" width="0" layer="19" extent="1-1"/>
-<wire x1="45.5" y1="40.6" x2="49.2" y2="43.0999" width="0" layer="19" extent="1-16"/>
-<wire x1="48.875" y1="36.375" x2="45.5" y2="34.7" width="0" layer="19" extent="1-16"/>
+<wire x1="45.76" y1="52.21" x2="57.625" y2="59.5" width="0" layer="19" extent="1-1"/>
+<wire x1="49.2" y1="43.0999" x2="45.5" y2="40.6" width="0" layer="19" extent="1-16"/>
 </signal>
 <signal name="+5V">
@@
 <contactref element="U7" pad="1"/>
 <contactref element="C6" pad="2"/>
-<contactref element="U6" pad="7"/>
-<contactref element="C8" pad="1"/>
-<wire x1="57.625" y1="55.3" x2="59.375" y2="63.7" width="0" layer="19" extent="1-1"/>
-<wire x1="50.15" y1="43.0999" x2="57.625" y2="55.3" width="0" layer="19" extent="1-1"/>
+<wire x1="50.15" y1="43.0999" x2="59.375" y2="63.7" width="0" layer="19" extent="1-1"/>
 <wire x1="48.25" y1="43.0999" x2="50.15" y2="43.0999" width="0" layer="19" extent="1-1"/>
-<wire x1="48.875" y1="41.025" x2="48.25" y2="43.0999" width="0" layer="19" extent="1-1"/>
-<wire x1="48" y1="30.2" x2="48.875" y2="41.025" width="0" layer="19" extent="1-1"/>
+<wire x1="48" y1="30.2" x2="48.25" y2="43.0999" width="0" layer="19" extent="1-1"/>
 <wire x1="47.55" y1="11.86" x2="47.6" y2="11.91" width="0" layer="19" extent="1-1"/>
 </signal>
@@
 <wire x1="33.6" y1="49.5" x2="30.5" y2="46.4" width="0.3" layer="16"/>
 <wire x1="30.5" y1="46.4" x2="29" y2="46.4" width="0.3" layer="16"/>
-<contactref element="U6" pad="5"/>
 <contactref element="TP2" pad="TP"/>
 <contactref element="R9" pad="2"/>
-<wire x1="43.6" y1="67.8" x2="59.45" y2="37.6" width="0" layer="19" extent="1-1"/>
-<wire x1="50.175" y1="41.025" x2="43.6" y2="67.8" width="0" layer="19" extent="1-1"/>
-<wire x1="24.8" y1="29.5" x2="50.175" y2="41.025" width="0" layer="19" extent="1-1"/>
+<wire x1="32.3" y1="61.0695" x2="43.6" y2="67.8" width="0" layer="19" extent="1-1"/>
+<wire x1="59.45" y1="37.6" x2="33.6" y2="49.5" width="0" layer="19" extent="1-16"/>
 </signal>
 <signal name="SWDIO">
@@
 <wire x1="40.8" y1="26.8" x2="36.7" y2="26.8" width="0.3" layer="1"/>
 <wire x1="44.79" y1="29.1" x2="44.81" y2="29.12" width="0.3" layer="1"/>
-<contactref element="U6" pad="1"/>
 <contactref element="R10" pad="1"/>
-<wire x1="48.225" y1="36.375" x2="48.85" y2="33.4" width="0" layer="19" extent="1-1"/>
-<wire x1="36.2" y1="27.3" x2="48.225" y2="36.375" width="0" layer="19" extent="1-1"/>
+<wire x1="44.81" y1="29.12" x2="48.85" y2="33.4" width="0" layer="19" extent="1-1"/>
 </signal>
 <signal name="PN_UART_TXD">
@@
 </signal>
 <signal name="+2V8">
-<contactref element="U6" pad="3"/>
 <contactref element="U7" pad="5"/>
 <contactref element="C7" pad="2"/>
-<contactref element="C9" pad="2"/>
-<contactref element="R7" pad="2"/>
-<wire x1="59.375" y1="51.1" x2="59.45" y2="42.4" width="0" layer="19" extent="1-1"/>
-<wire x1="59.375" y1="59.5" x2="59.375" y2="51.1" width="0" layer="19" extent="1-1"/>
-<wire x1="49.525" y1="36.375" x2="59.375" y2="59.5" width="0" layer="19" extent="1-1"/>
-<wire x1="48.25" y1="45.7001" x2="49.525" y2="36.375" width="0" layer="19" extent="1-1"/>
+<wire x1="48.25" y1="45.7001" x2="59.375" y2="59.5" width="0" layer="19" extent="1-1"/>
 </signal>
 <signal name="SWDCLK">
 <contactref element="U3" pad="6"/>
-<contactref element="U6" pad="8"/>
 <contactref element="R9" pad="1"/>
-<wire x1="48.225" y1="41.025" x2="57.75" y2="37.6" width="0" layer="19" extent="1-1"/>
-<wire x1="29.89" y1="23.48" x2="48.225" y2="41.025" width="0" layer="19" extent="1-1"/>
+<wire x1="29.89" y1="23.48" x2="57.75" y2="37.6" width="0" layer="19" extent="1-1"/>
 </signal>
 <signal name="PN_SWDIO">
-<contactref element="U6" pad="4"/>
 <contactref element="CONN1" pad="2"/>
 <contactref element="J3" pad="13"/>
 <contactref element="TP1" pad="TP"/>
 <contactref element="R10" pad="2"/>
+<wire x1="31.3" y1="61.0695" x2="39.5" y2="67.8" width="0" layer="19" extent="1-1"/>
 <wire x1="28.04" y1="49.068" x2="31.3" y2="61.0695" width="0" layer="19" extent="1-1"/>
-<wire x1="50.175" y1="36.375" x2="28.04" y2="49.068" width="0" layer="19" extent="1-1"/>
-<wire x1="39.5" y1="67.8" x2="50.175" y2="36.375" width="0" layer="19" extent="1-1"/>
-<wire x1="50.55" y1="33.4" x2="39.5" y2="67.8" width="0" layer="19" extent="1-1"/>
-</signal>
-<signal name="N$27">
-<contactref element="R7" pad="1"/>
-<contactref element="U6" pad="6"/>
-<contactref element="C10" pad="1"/>
-<wire x1="57.625" y1="46.9" x2="57.75" y2="42.4" width="0" layer="19" extent="1-1"/>
-<wire x1="49.525" y1="41.025" x2="57.625" y2="46.9" width="0" layer="19" extent="1-1"/>
+<wire x1="50.55" y1="33.4" x2="28.04" y2="49.068" width="0" layer="19" extent="1-1"/>
 </signal>
 </signals>

Commit message: Wrong suppressing of logical gates
Consider an error
Parts:
- removed C1, C2, C3: 100nF, rcl:C0603K
- removed C5: NC, rcl:C0603K
- removed JMP2: (no value), con-lstb:MA03-1
- removed R1: nc, resistor:R0603
- removed U1, U3, U4: TS5A9411, FabLib:SC70-6
- removed U5: SN74LVC1GU04DBV, 74LV:SOT23-5
Connections:
- removed net SWDO/RXD_1: JMP2.2, U4.4
- removed net SWDO/RXD_2: R1.2, U1.6, U4.6
- removed net SWD_EN: U3.1, U4.1, U5.4
- net +3V3: no longer C1.1, C2.1, C3.2, C5.2, U1.2, U3.2, U4.2, U5.5
- net FT_SWDCLK/TXD: no longer U3.5
- net FT_SWDI: no longer R1.1, U1.4
- net FT_SWDO/RXD: no longer U4.5
- net FT_SWD_EN_J2: no longer U5.2
- net FT_SWD_OE: no longer U1.1
- net GND: no longer C1.2, C2.2, C3.1, C5.1, U1.3, U3.3, U4.3, U5.3
- net PN_SWDO: no longer JMP2.1
- net PN_UART_RXD: no longer JMP2.3
- net PN_UART_TXD: no longer U3.4
- net SWDCLK: no longer U3.6
- net SWDIO: no longer U1.5
Routing:
- net SWD_EN: track 61.8 -> 0.00 mm, vias 3 -> 0
- net SWDIO: track 33.6 -> 0.00 mm
- net GND: track 184.9 -> 172.1 mm
- net PN_SWDO: track 85.3 -> 74.0 mm
- net +3V3: track 123.0 -> 113.6 mm
- net SWDO/RXD_2: track 9.28 -> 0.00 mm, vias 2 -> 0
- net SWDO/RXD_1: track 7.06 -> 0.00 mm
- net FT_SWDI: track 16.0 -> 9.62 mm
- net FT_SWDCLK/TXD: track 8.88 -> 5.26 mm
- net FT_SWD_EN_J2: track 9.22 -> 7.92 mm
- net PN_UART_RXD: track 95.5 -> 94.4 mm
- net FT_SWDO/RXD: track 12.1 -> 11.1 mm
- net PN_UART_TXD: track 54.5 -> 53.8 mm
